Commit message: Mapping my World

File: my_robot/urdf/my_robot.xacro (robot description, xacro)
@@ -2,4 +2,11 @@
   <xacro:include filename="$(find my_robot)/urdf/my_robot.gazebo" />
   <link name="robot_footprint"></link>
+ <joint name="camera_optical_joint" type="fixed">
+  <origin xyz="0 0 0" rpy="-1.5705 0 -1.5707"/>
+  <parent link="camera"/>
+  <child link="camera_link_optical"/>
+ </joint>
+ <link name="camera_link_optical">
+ </link>
   <link name='camera'>
     <inertial>
